Commit message: updated kinova_common.xacro for bramblebee's custom end effector

File: kinova_description/urdf/kinova_common.xacro (robot description, xacro)
@@ -15,10 +15,16 @@
 <xacro:include filename="$(find kinova_description)/urdf/kinova_inertial.xacro" />
     <xacro:property name="J_PI" value="3.1415926535897931" />
-    <xacro:macro name="kinova_armlink" params="link_name link_mesh ring_mesh:=ring_big use_ring_mesh:=false mesh_no">
+    <xacro:macro name="kinova_armlink" params="link_name link_mesh ring_mesh:=ring_big use_ring_mesh:=false mesh_no custom_link:=false">
         <link name="${link_name}">
             <visual>
                 <geometry>
+									<xacro:if value="${custom_link}">
+                    <mesh
+                        filename="package://manipulation_description/meshes/${link_mesh}.dae"/>
+									</xacro:if>
+									<xacro:unless value="${custom_link}">
                     <mesh
                         filename="package://kinova_description/meshes/${link_mesh}.dae"/>
+									</xacro:if>
                 </geometry>
                 <material name="carbon_fiber">
@@ -37,6 +43,12 @@
             <collision>
                 <geometry>
+									<xacro:if value="${custom_link}">
+                    <mesh
+                        filename="package://manipulation_description/meshes/${link_mesh}.dae"/>
+									</xacro:if>
+									<xacro:unless value="${custom_link}">
                     <mesh
                         filename="package://kinova_description/meshes/${link_mesh}.dae"/>
+									</xacro:if>
                 </geometry>
             </collision>
